Commit message: Changes to roundbot - Changed laser to LDLidar - Update base - Moved ball casters

File: andino_description/urdf/include/common_sensors.urdf.xacro (robot description, xacro)
@@ -9,5 +9,5 @@
       <origin xyz="0 0 0" rpy="0 0 ${pi}"/>
       <geometry>
-        <mesh filename="package://andino_description/meshes/sensors/${mesh}" />
+        <mesh filename="package://andino_description/meshes/sensors/${mesh}" scale="0.001 0.001 0.001" />
       </geometry>
       <material name="dark_grey"/>
@@ -38,5 +38,5 @@
     <parent link="${parent_link}"/>
     <child link="${prefix}_laser_link"/>
-    <origin xyz="${sensor_prop['laser']['dx']} ${sensor_prop['laser']['dy']} ${sensor_prop['laser']['dz']}" rpy="0 0 ${pi}"/>
+    <origin xyz="${sensor_prop['laser']['dx']} ${sensor_prop['laser']['dy']} ${sensor_prop['laser']['dz']}" rpy="0 0 0"/>
     <axis xyz="0 1 0" />
   </joint>

File: andino_description/urdf/roundbot/andino.urdf.xacro (robot description, xacro)
@@ -24,5 +24,5 @@
               mesh="${base_props['base']['mesh']}"
               scale="${base_props['base']['scale']}">
-        <origin xyz="-0.11 -0.11 -0.12" rpy="0 0 0" />
+        <origin xyz="0 0 -0.045" rpy="0 0 0" />
   </xacro:base>
   <!-- Caster Wheel -->

File: andino_description/urdf/roundbot/caster_macro.urdf.xacro (robot description, xacro)
@@ -20,5 +20,5 @@
                           r="${caster_props['base']['size']['diameter'] / 2}"/>
       <visual>
-        <origin xyz="-0.11 0.11 0.0085" rpy="${pi} 0 0" />
+        <origin xyz="-0.11 0.11 0.0073" rpy="${pi} 0 0" />
         <geometry>
             <mesh filename="package://andino_description/meshes/${robot_name}/${caster_props['base']['mesh']}" scale="${scale}"/>
@@ -27,5 +27,5 @@
       </visual>
       <collision>
-        <origin xyz="0 0 -0.006" rpy="0 0 0" />
+        <origin xyz="0 0 -0.0066" rpy="0 0 0" />
         <geometry>
           <sphere radius="${caster_props['base']['size']['diameter'] / 2}" />
